File: Card template/project.kicad_pcb (KiCad board)
At the start: 2 copper layers, 48.5 x 20 mm, 3 parts, among them U1 24LC32, X0 Card Edge

Commit message: updates
Other:
- board text added: "github.com/aspro648/RPB"
Changed lines of the file:
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@@
   (general
     (thickness 1.6)
-    (drawings 6)
+    (drawings 7)
     (tracks 120)
     (zones 0)
@@
       (net 24 +5V))
   )
+  (gr_text github.com/aspro648/RPB (at 27 -1.5) (layer B.SilkS)
+    (effects (font (size 0.8 0.8) (thickness 0.15) italic) (justify mirror))
+  )
   (gr_line (start 9.75 -19.5) (end 9.75 -0.5) (layer Dwgs.User) (width 0.15))
-  (gr_text Template (at 28.25 -2) (layer F.SilkS)
+  (gr_text Template (at 27.5 -2) (layer F.SilkS)
     (effects (font (size 1.5 1.5) (thickness 0.25) italic))
   )
-  (gr_text "Rapid Prototyping Card" (at 27.75 -2) (layer B.SilkS)
+  (gr_text "Rapid Prototyping Card" (at 27 -3) (layer B.SilkS)
     (effects (font (size 1 1) (thickness 0.25) italic) (justify mirror))
   )
