File: Card template/project.sch (KiCad schematic (older format))
At the start: 7 parts, among them J1 Molex PicoBlade, J2 Hirose DF13, J3 TestPoints, J4 TestPoints, U1 24LC32, X0 Card Edge

Commit message: EEPROM footprint update
Parts:
- U1: footprint Package_DFN_QFN:DFN-8-1EP_2x3mm_P0.5mm_EP0.61x2.2mm -> footprints:DFN-8-1EP_3x2mm
Connections:
- no-connect marks 1 -> 2
Changed lines of the file:
@@
 F 0 "U1" H 1900 7100 50  0000 C CNN
 F 1 "24LC32" H 2350 6550 50  0000 C CNN
-F 2 "Package_DFN_QFN:DFN-8-1EP_2x3mm_P0.5mm_EP0.61x2.2mm" H 2100 6850 50  0001 C CNN
+F 2 "footprints:DFN-8-1EP_3x2mm" H 2100 6850 50  0001 C CNN
 F 3 "http://ww1.microchip.com/downloads/en/DeviceDoc/21072G.pdf" H 2100 6850 50  0001 C CNN
 	1    2100 6850
@@
 	1    0    0    -1
 $EndComp
+NoConn ~ 3350 4150
 $EndSCHEMATC
