File: Card 254mm/project.sch (KiCad schematic (older format))
At the start: 9 parts, among them J1 Conn_01x04, J2 Conn_01x10, J3 Conn_01x10, J4 Conn_01x10, J5 Conn_01x10, J6 Conn_01x10, U1 24LC32, X0 Card Edge

Commit message: EEPROM footprint update
Parts:
- U1: footprint Package_DFN_QFN:DFN-8-1EP_2x3mm_P0.5mm_EP0.61x2.2mm -> footprints:DFN-8-1EP_3x2mm
Changed lines of the file:
@@
 F 0 "U1" H 1900 7100 50  0000 C CNN
 F 1 "24LC32" H 2350 6550 50  0000 C CNN
-F 2 "Package_DFN_QFN:DFN-8-1EP_2x3mm_P0.5mm_EP0.61x2.2mm" H 2100 6850 50  0001 C CNN
+F 2 "footprints:DFN-8-1EP_3x2mm" H 2100 6850 50  0001 C CNN
 F 3 "http://ww1.microchip.com/downloads/en/DeviceDoc/21072G.pdf" H 2100 6850 50  0001 C CNN
 	1    2100 6850

Commit message: updates
Changed lines of the file:
@@
-$EndComp
-$Comp
-L project:+5V #PWR0110
-U 1 1 638338CD
-P 4650 5050
-F 0 "#PWR0110" H 4650 4900 50  0001 C CNN
-F 1 "+5V" H 4650 5190 50  0000 C CNN
-F 2 "" H 4650 5050 50  0001 C CNN
-F 3 "" H 4650 5050 50  0001 C CNN
-	1    4650 5050
-	0    -1   -1   0
 $EndComp
 $Comp
 L project:GND #PWR0111
 U 1 1 63833D6C
-P 4650 5150
-F 0 "#PWR0111" H 4650 4900 50  0001 C CNN
-F 1 "GND" H 4650 5000 50  0000 C CNN
-F 2 "" H 4650 5150 50  0001 C CNN
-F 3 "" H 4650 5150 50  0001 C CNN
-	1    4650 5150
+P 4650 5050
+F 0 "#PWR0111" H 4650 4800 50  0001 C CNN
+F 1 "GND" H 4650 4900 50  0000 C CNN
+F 2 "" H 4650 5050 50  0001 C CNN
+F 3 "" H 4650 5050 50  0001 C CNN
+	1    4650 5050
 	0    1    1    0
 $EndComp
@@
 	1    0    0    -1
 $EndComp
+$Comp
+L project:+5V #PWR0110
+U 1 1 638338CD
+P 4650 5150
+F 0 "#PWR0110" H 4650 5000 50  0001 C CNN
+F 1 "+5V" H 4650 5290 50  0000 C CNN
+F 2 "" H 4650 5150 50  0001 C CNN
+F 3 "" H 4650 5150 50  0001 C CNN
+	1    4650 5150
+	0    -1   -1   0
+$EndComp
+Text Label 5600 4150 0    60   ~ 0
+D3_SCL
 $EndSCHEMATC
