File: Board/project.sch (KiCad schematic (older format))
At the start: 77 parts, among them J1 USB_OTG, J2 ISP, P1 M3, P2 M3, P3 M3, P4 M3, P5 Standoff, P6 Standoff, SW1 RESET, SW2 SCK, U1 ATMEGA32U4-AU, X1 MEC8-113, X2 MEC8-113, Y1 16 Mhz

Commit message: updates
Parts:
- renumbered R29 to R27
Changed lines of the file:
@@
 Comment4 ""
 $EndDescr
-$Comp
-L project:ATMEGA32U4-AU U1
-U 1 1 5B3FD92A
-P 7400 2850
-F 0 "U1" H 6450 4550 50  0000 C CNN
-F 1 "ATMEGA32U4-AU" H 8100 1350 50  0000 C CNN
-F 2 "footprints:TQFP-44_10x10mm_Pitch0.8mm" H 7400 2850 50  0001 C CIN
-F 3 "" H 8500 3950 50  0001 C CNN
-	1    7400 2850
-	1    0    0    -1
-$EndComp
 Text Label 8650 1400 0    60   ~ 0
 SCK
@@
 	8500 1600 8800 1600
 Wire Wire Line
-	8500 1700 8800 1700
-Wire Wire Line
 	8500 1800 8800 1800
 Wire Wire Line
@@
 Wire Wire Line
 	8500 4200 8800 4200
-Wire Wire Line
-	7000 4450 7250 4450
-Connection ~ 7450 4450
-Connection ~ 7350 4450
-Connection ~ 7250 4450
 Connection ~ 7300 4450
-Connection ~ 7550 1050
-Connection ~ 7300 1050
 Connection ~ 7400 1050
 Wire Wire Line
@@
 Wire Wire Line
 	3200 2750 3200 2850
-Wire Wire Line
-	7200 1050 7300 1050
 Connection ~ 5100 2650
 Wire Wire Line
@@
 	5850 1650 6050 1650
 Connection ~ 6050 1650
-Wire Wire Line
-	7450 4450 7550 4450
-Wire Wire Line
-	7350 4450 7450 4450
-Wire Wire Line
-	7250 4450 7300 4450
-Wire Wire Line
-	7300 4450 7350 4450
-Wire Wire Line
-	7550 1050 7650 1050
-Wire Wire Line
-	7300 1050 7400 1050
-Wire Wire Line
-	7400 1050 7550 1050
 Wire Wire Line
 	6100 2900 6250 2900
@@
 $EndComp
 $Comp
-L project:R R29
-U 1 1 63C58743
-P 2700 6200
-F 0 "R29" V 2750 6000 50  0000 C CNN
-F 1 "4K7" V 2700 6200 50  0000 C CNN
-F 2 "footprints:R_0603" V 2630 6200 50  0001 C CNN
-F 3 "" H 2700 6200 50  0001 C CNN
-	1    2700 6200
-	0    -1   -1   0
-$EndComp
-$Comp
 L project:+5V #PWR0112
 U 1 1 63C588C4
@@
 Connection ~ 1450 6300
 $Comp
-L project:GND #PWR?
+L project:GND #PWR0110
 U 1 1 63F8BC64
 P 4800 6300
-F 0 "#PWR?" H 4800 6050 50  0001 C CNN
+F 0 "#PWR0110" H 4800 6050 50  0001 C CNN
 F 1 "GND" H 4800 6150 50  0000 C CNN
 F 2 "" H 4800 6300 50  0001 C CNN
@@
 	0    1    1    0
 $EndComp
+$Comp
+L project:R R27
+U 1 1 63C58743
+P 2700 6200
+F 0 "R27" V 2750 6000 50  0000 C CNN
+F 1 "4K7" V 2700 6200 50  0000 C CNN
+F 2 "footprints:R_0603" V 2630 6200 50  0001 C CNN
+F 3 "" H 2700 6200 50  0001 C CNN
+	1    2700 6200
+	0    -1   -1   0
+$EndComp
+Wire Wire Line
+	7400 1050 7550 1050
+Wire Wire Line
+	7550 1050 7650 1050
+Wire Wire Line
+	7300 4450 7350 4450
+Wire Wire Line
+	7350 4450 7450 4450
+Wire Wire Line
+	7450 4450 7550 4450
+Wire Wire Line
+	7300 1050 7400 1050
+Wire Wire Line
+	7200 1050 7300 1050
+Connection ~ 7300 1050
+Connection ~ 7550 1050
+Connection ~ 7250 4450
+Connection ~ 7350 4450
+Connection ~ 7450 4450
+Wire Wire Line
+	7250 4450 7300 4450
+Wire Wire Line
+	7000 4450 7250 4450
+Wire Wire Line
+	8500 1700 8800 1700
+$Comp
+L project:ATMEGA32U4-AU U1
+U 1 1 5B3FD92A
+P 7400 2850
+F 0 "U1" H 6450 4550 50  0000 C CNN
+F 1 "ATMEGA32U4-AU" H 8100 1350 50  0000 C CNN
+F 2 "footprints:TQFP-44_10x10mm_Pitch0.8mm" H 7400 2850 50  0001 C CIN
+F 3 "" H 8500 3950 50  0001 C CNN
+	1    7400 2850
+	1    0    0    -1
+$EndComp
 $EndSCHEMATC

Commit message: Updates
Parts:
- removed SnakeBack1, SnakeFront1: SYM_Arrow_Large, footprints:Snake, symbol Graphic:SYM_Arrow_Large
- added C2: 0.1uF, footprints:C_0603, symbol project:C
- added JP1: JMP, footprints:Jumper, symbol Device:Jumper_NO_Small
- added R29: 0.1, footprints:R_1206, symbol Device:R
- added U2: INA219AxD, Package_SO:SOIC-8_3.9x4.9mm_P1.27mm, symbol Analog_ADC:INA219AxD
Connections:
- net labels added: SYM_Arrow_Large, Vin
- wire segments 215 -> 241
- no-connect marks 5 -> 4
Other:
- note added: "i2c: 0x40"
- moved on the sheet: F1
Changed lines of the file:
@@
 L project:Polyfuse F1
 U 1 1 5B6E44FA
-P 5750 2450
-F 0 "F1" V 5650 2350 50  0000 C CNN
-F 1 "Polyfuse" V 5800 2600 50  0000 C CNN
-F 2 "footprints:R_0805_HandSoldering" H 5800 2250 50  0001 L CNN
-F 3 "" H 5750 2450 50  0001 C CNN
-	1    5750 2450
-	0    1    1    0
-$EndComp
-NoConn ~ 5750 2450
+P 5150 2450
+F 0 "F1" V 5050 2350 50  0000 C CNN
+F 1 "Polyfuse" V 5200 2600 50  0000 C CNN
+F 2 "footprints:R_0805_HandSoldering" H 5200 2250 50  0001 L CNN
+F 3 "" H 5150 2450 50  0001 C CNN
+	1    5150 2450
+	0    1    1    0
+$EndComp
 $Comp
 L project:VBUS #PWR016
@@
 	6100 2500 6250 2500
 Wire Wire Line
-	6100 2500 6100 2450
-Wire Wire Line
 	6250 2650 5950 2650
 Wire Wire Line
@@
 Wire Wire Line
 	4900 2750 5350 2750
-Wire Wire Line
-	4900 2450 5600 2450
-Wire Wire Line
-	6100 2450 5900 2450
 Wire Wire Line
 	9350 3500 9350 3450
@@
 	1    0    0    -1
 $EndComp
-Wire Wire Line
-	6100 2450 6100 2400
-Connection ~ 6100 2450
 $Comp
 L project:R R1
@@
 $EndComp
 $Comp
-L Graphic:SYM_Arrow_Large SnakeFront1
+L Graphic:SYM_Arrow_Large #SnakeFront1
 U 1 1 6390CCB5
 P 2950 7650
-F 0 "SnakeFront1" H 2946 7753 50  0000 C CNN
+F 0 "#SnakeFront1" H 2946 7753 50  0000 C CNN
 F 1 "SYM_Arrow_Large" H 2950 7570 50  0001 C CNN
 F 2 "footprints:Snake" H 2950 7650 50  0001 C CNN
@@
 $EndComp
 $Comp
-L Graphic:SYM_Arrow_Large SnakeBack1
+L Graphic:SYM_Arrow_Large #SnakeBack1
 U 1 1 6390D071
 P 2950 7850
-F 0 "SnakeBack1" H 2946 7953 50  0000 C CNN
+F 0 "#SnakeBack1" H 2946 7953 50  0000 C CNN
 F 1 "SYM_Arrow_Large" H 2950 7770 50  0001 C CNN
 F 2 "footprints:Snake" H 2950 7850 50  0001 C CNN
@@
 	1    0    0    -1
 $EndComp
+$Comp
+L Analog_ADC:INA219AxD U2
+U 1 1 638CCFE0
+P 8400 5650
+F 0 "U2" H 8200 6000 50  0000 C CNN
+F 1 "INA219AxD" H 8050 5250 50  0000 C CNN
+F 2 "Package_SO:SOIC-8_3.9x4.9mm_P1.27mm" H 9200 5300 50  0001 C CNN
+F 3 "http://www.ti.com/lit/ds/symlink/ina219.pdf" H 8750 5550 50  0001 C CNN
+	1    8400 5650
+	1    0    0    -1
+$EndComp
+$Comp
+L project:GND #PWR0115
+U 1 1 638CEDC3
+P 8400 6150
+F 0 "#PWR0115" H 8400 5900 50  0001 C CNN
+F 1 "GND" H 8400 6000 50  0000 C CNN
+F 2 "" H 8400 6150 50  0001 C CNN
+F 3 "" H 8400 6150 50  0001 C CNN
+	1    8400 6150
+	1    0    0    -1
+$EndComp
+Wire Wire Line
+	8000 5750 7900 5750
+Wire Wire Line
+	8400 6100 8400 6050
+Wire Wire Line
+	8400 6100 8400 6150
+Connection ~ 8400 6100
+Wire Wire Line
+	8800 5750 9000 5750
+Wire Wire Line
+	9000 5750 9000 5850
+Wire Wire Line
+	9000 6100 8400 6100
+Wire Wire Line
+	8750 5850 8800 5850
+Connection ~ 9000 5850
+Wire Wire Line
+	9000 5850 9000 6100
+Connection ~ 8800 5850
+Wire Wire Line
+	8800 5850 9000 5850
+Wire Wire Line
+	8800 5450 9200 5450
+Wire Wire Line
+	8800 5550 9200 5550
+Text Label 8900 5550 0    60   ~ 0
+D3_SCL
+Text Label 8850 5450 0    60   ~ 0
+D2_SDA
+$Comp
+L Device:R R29
+U 1 1 63942558
+P 7650 5650
+F 0 "R29" H 7720 5696 50  0000 L CNN
+F 1 "0.1" H 7720 5605 50  0000 L CNN
+F 2 "footprints:R_1206" V 7580 5650 50  0001 C CNN
+F 3 "~" H 7650 5650 50  0001 C CNN
+	1    7650 5650
+	1    0    0    -1
+$EndComp
+Wire Wire Line
+	6100 2400 6100 2500
+Wire Wire Line
+	4900 2450 5000 2450
+Wire Wire Line
+	5300 2450 5650 2450
+Text Label 5450 2450 0    60   ~ 0
+Vin
+Wire Wire Line
+	7900 5750 7900 5900
+Wire Wire Line
+	7900 5900 7650 5900
+Wire Wire Line
+	7650 5900 7650 5800
+Wire Wire Line
+	8000 5550 7900 5550
+Wire Wire Line
+	7900 5550 7900 5350
+Wire Wire Line
+	7900 5350 7650 5350
+Wire Wire Line
+	7650 5350 7650 5500
+Wire Wire Line
+	7650 5900 7450 5900
+Connection ~ 7650 5900
+Text Label 7200 5900 0    60   ~ 0
+Vin
+$Comp
+L project:+5V #PWR0116
+U 1 1 63B23406
+P 7650 5200
+F 0 "#PWR0116" H 7650 5050 50  0001 C CNN
+F 1 "+5V" H 7650 5340 50  0000 C CNN
+F 2 "" H 7650 5200 50  0001 C CNN
+F 3 "" H 7650 5200 50  0001 C CNN
+	1    7650 5200
+	1    0    0    -1
+$EndComp
+$Comp
+L project:+5V #PWR0117
+U 1 1 63B23B58
+P 8400 5200
+F 0 "#PWR0117" H 8400 5050 50  0001 C CNN
+F 1 "+5V" H 8400 5340 50  0000 C CNN
+F 2 "" H 8400 5200 50  0001 C CNN
+F 3 "" H 8400 5200 50  0001 C CNN
+	1    8400 5200
+	1    0    0    -1
+$EndComp
+$Comp
+L project:+5V #PWR0118
+U 1 1 63B24080
+P 9400 5200
+F 0 "#PWR0118" H 9400 5050 50  0001 C CNN
+F 1 "+5V" H 9400 5340 50  0000 C CNN
+F 2 "" H 9400 5200 50  0001 C CNN
+F 3 "" H 9400 5200 50  0001 C CNN
+	1    9400 5200
+	1    0    0    -1
+$EndComp
+$Comp
+L project:GND #PWR0119
+U 1 1 63B244C9
+P 9400 6100
+F 0 "#PWR0119" H 9400 5850 50  0001 C CNN
+F 1 "GND" H 9400 5950 50  0000 C CNN
+F 2 "" H 9400 6100 50  0001 C CNN
+F 3 "" H 9400 6100 50  0001 C CNN
+	1    9400 6100
+	1    0    0    -1
+$EndComp
+$Comp
+L project:C C2
+U 1 1 63B24868
+P 9400 5650
+F 0 "C2" H 9425 5750 50  0000 L CNN
+F 1 "0.1uF" H 9425 5550 50  0000 L CNN
+F 2 "footprints:C_0603" H 9438 5500 50  0001 C CNN
+F 3 "" H 9400 5650 50  0001 C CNN
+	1    9400 5650
+	1    0    0    -1
+$EndComp
+Wire Wire Line
+	9400 6100 9400 5800
+Wire Wire Line
+	9400 5500 9400 5200
+Wire Wire Line
+	8400 5250 8400 5200
+Wire Wire Line
+	7650 5350 7650 5200
+Connection ~ 7650 5350
+$Comp
+L Device:Jumper_NO_Small JP1
+U 1 1 63B76AE5
+P 7450 5650
+F 0 "JP1" V 7400 5450 50  0000 L CNN
+F 1 "JMP" V 7500 5450 50  0000 L CNN
+F 2 "footprints:Jumper" H 7450 5650 50  0001 C CNN
+F 3 "~" H 7450 5650 50  0001 C CNN
+	1    7450 5650
+	0    1    1    0
+$EndComp
+Wire Wire Line
+	7450 5900 7450 5750
+Connection ~ 7450 5900
+Wire Wire Line
+	7450 5900 7150 5900
+Wire Wire Line
+	7450 5550 7450 5350
+Wire Wire Line
+	7450 5350 7650 5350
+Text Notes 7850 6200 0    60   ~ 0
+i2c: 0x40
 $EndSCHEMATC

Commit message: updates
Parts:
- added SnakeBack1: SYM_Arrow_Large, footprints:Snake, symbol Graphic:SYM_Arrow_Large
- CardOutline1, CardOutline2: footprint footprints:MEC8-113-CARD-OUTLINE -> footprints:MEC8-113-CARD_2outline
Changed lines of the file:
@@
 F 0 "CardOutline1" H 2346 7753 50  0000 C CNN
 F 1 "SYM_Arrow_Large" H 2350 7570 50  0001 C CNN
-F 2 "footprints:MEC8-113-CARD-OUTLINE" H 2350 7650 50  0001 C CNN
+F 2 "footprints:MEC8-113-CARD_2outline" H 2350 7650 50  0001 C CNN
 F 3 "~" H 2350 7650 50  0001 C CNN
 	1    2350 7650
@@
 F 0 "CardOutline2" H 2346 7953 50  0000 C CNN
 F 1 "SYM_Arrow_Large" H 2350 7770 50  0001 C CNN
-F 2 "footprints:MEC8-113-CARD-OUTLINE" H 2350 7850 50  0001 C CNN
+F 2 "footprints:MEC8-113-CARD_2outline" H 2350 7850 50  0001 C CNN
 F 3 "~" H 2350 7850 50  0001 C CNN
 	1    2350 7850
@@
 $EndComp
 $Comp
-L Graphic:SYM_Arrow_Large #SnakeBack1
+L Graphic:SYM_Arrow_Large SnakeBack1
 U 1 1 6390D071
 P 2950 7850
-F 0 "#SnakeBack1" H 2946 7953 50  0000 C CNN
+F 0 "SnakeBack1" H 2946 7953 50  0000 C CNN
 F 1 "SYM_Arrow_Large" H 2950 7770 50  0001 C CNN
 F 2 "footprints:Snake" H 2950 7850 50  0001 C CNN

Commit message: Updates
Parts:
- added R30: 1K, footprints:R_0603, symbol project:R
- added U3: 24LC32, footprints:DFN-8-1EP_3x2mm, symbol Memory_EEPROM:24LC32
Connections:
- no-connect marks 4 -> 11
Other:
- note added: "For card stencil"
- moved on the sheet: CardOutline1, CardOutline2, MadeInOregon1, MadeWithKiCAD1, OSHW1, SnakeBack1
Changed lines of the file:
@@
 L Graphic:SYM_Arrow_Large CardOutline1
 U 1 1 63747108
-P 2350 7650
-F 0 "CardOutline1" H 2346 7753 50  0000 C CNN
-F 1 "SYM_Arrow_Large" H 2350 7570 50  0001 C CNN
-F 2 "footprints:MEC8-113-CARD_2outline" H 2350 7650 50  0001 C CNN
-F 3 "~" H 2350 7650 50  0001 C CNN
-	1    2350 7650
+P 3900 7600
+F 0 "CardOutline1" H 3896 7703 50  0000 C CNN
+F 1 "SYM_Arrow_Large" H 3900 7520 50  0001 C CNN
+F 2 "footprints:MEC8-113-CARD_2outline" H 3900 7600 50  0001 C CNN
+F 3 "~" H 3900 7600 50  0001 C CNN
+	1    3900 7600
 	1    0    0    -1
 $EndComp
@@
 L Graphic:SYM_Arrow_Large CardOutline2
 U 1 1 63748B06
-P 2350 7850
-F 0 "CardOutline2" H 2346 7953 50  0000 C CNN
-F 1 "SYM_Arrow_Large" H 2350 7770 50  0001 C CNN
-F 2 "footprints:MEC8-113-CARD_2outline" H 2350 7850 50  0001 C CNN
-F 3 "~" H 2350 7850 50  0001 C CNN
-	1    2350 7850
+P 3900 7800
+F 0 "CardOutline2" H 3896 7903 50  0000 C CNN
+F 1 "SYM_Arrow_Large" H 3900 7720 50  0001 C CNN
+F 2 "footprints:MEC8-113-CARD_2outline" H 3900 7800 50  0001 C CNN
+F 3 "~" H 3900 7800 50  0001 C CNN
+	1    3900 7800
 	1    0    0    -1
 $EndComp
@@
 L Graphic:SYM_Arrow_Large #SnakeFront1
 U 1 1 6390CCB5
-P 2950 7650
-F 0 "#SnakeFront1" H 2946 7753 50  0000 C CNN
-F 1 "SYM_Arrow_Large" H 2950 7570 50  0001 C CNN
-F 2 "footprints:Snake" H 2950 7650 50  0001 C CNN
-F 3 "~" H 2950 7650 50  0001 C CNN
-	1    2950 7650
+P 4500 7600
+F 0 "#SnakeFront1" H 4496 7703 50  0000 C CNN
+F 1 "SYM_Arrow_Large" H 4500 7520 50  0001 C CNN
+F 2 "footprints:Snake" H 4500 7600 50  0001 C CNN
+F 3 "~" H 4500 7600 50  0001 C CNN
+	1    4500 7600
 	1    0    0    -1
 $EndComp
@@
 L Graphic:SYM_Arrow_Large SnakeBack1
 U 1 1 6390D071
-P 2950 7850
-F 0 "SnakeBack1" H 2946 7953 50  0000 C CNN
-F 1 "SYM_Arrow_Large" H 2950 7770 50  0001 C CNN
-F 2 "footprints:Snake" H 2950 7850 50  0001 C CNN
-F 3 "~" H 2950 7850 50  0001 C CNN
-	1    2950 7850
+P 4500 7800
+F 0 "SnakeBack1" H 4496 7903 50  0000 C CNN
+F 1 "SYM_Arrow_Large" H 4500 7720 50  0001 C CNN
+F 2 "footprints:Snake" H 4500 7800 50  0001 C CNN
+F 3 "~" H 4500 7800 50  0001 C CNN
+	1    4500 7800
 	1    0    0    -1
 $EndComp
@@
 L Graphic:SYM_Arrow_Large MadeWithKiCAD1
 U 1 1 63AF2EFE
-P 3500 7650
-F 0 "MadeWithKiCAD1" H 3496 7753 50  0000 C CNN
-F 1 "SYM_Arrow_Large" H 3500 7570 50  0001 C CNN
-F 2 "footprints:KiCad-Logo2_8mm_SilkScreen" H 3500 7650 50  0001 C CNN
-F 3 "~" H 3500 7650 50  0001 C CNN
-	1    3500 7650
+P 5050 7600
+F 0 "MadeWithKiCAD1" H 5046 7703 50  0000 C CNN
+F 1 "SYM_Arrow_Large" H 5050 7520 50  0001 C CNN
+F 2 "footprints:KiCad-Logo2_8mm_SilkScreen" H 5050 7600 50  0001 C CNN
+F 3 "~" H 5050 7600 50  0001 C CNN
+	1    5050 7600
 	1    0    0    -1
 $EndComp
@@
 L Graphic:SYM_Arrow_Large OSHW1
 U 1 1 63AF328A
-P 3500 7850
-F 0 "OSHW1" H 3496 7953 50  0000 C CNN
-F 1 "SYM_Arrow_Large" H 3500 7770 50  0001 C CNN
-F 2 "footprints:OSHW-Logo_11.4x12mm_SilkScreen" H 3500 7850 50  0001 C CNN
-F 3 "~" H 3500 7850 50  0001 C CNN
-	1    3500 7850
+P 5050 7800
+F 0 "OSHW1" H 5046 7903 50  0000 C CNN
+F 1 "SYM_Arrow_Large" H 5050 7720 50  0001 C CNN
+F 2 "footprints:OSHW-Logo_11.4x12mm_SilkScreen" H 5050 7800 50  0001 C CNN
+F 3 "~" H 5050 7800 50  0001 C CNN
+	1    5050 7800
 	1    0    0    -1
 $EndComp
@@
 L Graphic:SYM_Arrow_Large MadeInOregon1
 U 1 1 63AF35D1
-P 4000 7850
-F 0 "MadeInOregon1" H 3996 7953 50  0000 C CNN
-F 1 "SYM_Arrow_Large" H 4000 7770 50  0001 C CNN
-F 2 "footprints:MadeInOregonRev25" H 4000 7850 50  0001 C CNN
-F 3 "~" H 4000 7850 50  0001 C CNN
-	1    4000 7850
+P 5550 7800
+F 0 "MadeInOregon1" H 5546 7903 50  0000 C CNN
+F 1 "SYM_Arrow_Large" H 5550 7720 50  0001 C CNN
+F 2 "footprints:MadeInOregonRev25" H 5550 7800 50  0001 C CNN
+F 3 "~" H 5550 7800 50  0001 C CNN
+	1    5550 7800
 	1    0    0    -1
 $EndComp
@@
 Text Notes 7850 6200 0    60   ~ 0
 i2c: 0x40
+$Comp
+L Memory_EEPROM:24LC32 U3
+U 1 1 63911A51
+P 1700 7500
+F 0 "U3" H 1500 7750 50  0000 C CNN
+F 1 "24LC32" H 1900 7750 50  0000 C CNN
+F 2 "footprints:DFN-8-1EP_3x2mm" H 1700 7500 50  0001 C CNN
+F 3 "http://ww1.microchip.com/downloads/en/DeviceDoc/21072G.pdf" H 1700 7500 50  0001 C CNN
+	1    1700 7500
+	1    0    0    -1
+$EndComp
+$Comp
+L project:R R30
+U 1 1 63912A10
+P 2300 7500
+F 0 "R30" V 2380 7500 50  0000 C CNN
+F 1 "1K" V 2300 7500 50  0000 C CNN
+F 2 "footprints:R_0603" V 2230 7500 50  0001 C CNN
+F 3 "" H 2300 7500 50  0001 C CNN
+	1    2300 7500
+	1    0    0    -1
+$EndComp
+Text Notes 1550 7900 0    60   ~ 0
+For card stencil
+NoConn ~ 1300 7400
+NoConn ~ 1300 7500
+NoConn ~ 1300 7600
+NoConn ~ 1700 7800
+NoConn ~ 1700 7200
+NoConn ~ 2300 7350
+NoConn ~ 2300 7650
+Wire Notes Line
+	1150 7100 2500 7100
+Wire Notes Line
+	2500 7100 2500 7950
+Wire Notes Line
+	2500 7950 1150 7950
+Wire Notes Line
+	1150 7950 1150 7100
 $EndSCHEMATC
