File: Board/project.kicad_pcb (KiCad board)
At the start: 2 copper layers, 64.8 x 50.8 mm, 77 parts, among them J1 USB_OTG, J2 ISP, P1 M3, P2 M3, P3 M3, P4 M3, P5 Standoff, P6 Standoff, SW1 RESET, SW2 SCK, U1 ATMEGA32U4-AU, X1 MEC8-113, X2 MEC8-113, Y1 16 Mhz

Commit message: updates
Parts:
- renumbered R29 to R27
Other:
- board text added: "Keep It Simple Stupid"
- board text added: "github.com/aspro648/RPB"

Commit message: Updates
Parts:
- removed SnakeBack1, SnakeFront1: SYM_Arrow_Large, footprints:Snake
- added C2: 0.1uF, footprints:C_0603, F.Cu at (157.0, 103.5)
- added JP1: JMP, footprints:Jumper, F.Cu at (151.5, 106.8)
- added R29: 0.1, footprints:R_1206, F.Cu at (151.5, 106.8)
- added U2: INA219AxD, Package_SO:SOIC-8_3.9x4.9mm_P1.27mm, F.Cu at (157.0, 107.5)
- moved P5 3.00 mm to (168.0, 88.0)
- moved P6 2.90 mm to (168.0, 110.0)
Connections:
- F1 pad 1: +5V -> /Vin
Routing:
- net /Vin: track 0.00 -> 105.1 mm, vias 0 -> 2
- net GND: track 283.1 -> 231.7 mm
- net /D2_SDA: track 115.4 -> 134.3 mm, vias 4 -> 5
- net /D3_SCL: track 117.3 -> 135.5 mm, vias 4 -> 5
- net +5V: track 238.6 -> 250.4 mm, vias 10 -> 9
- net /D0: track 115.7 -> 119.2 mm
- net Net-(D23-Pad1): track 24.4 -> 25.6 mm
Other:
- board text added: "0x40"

Commit message: updates
Parts:
- added SnakeBack1: SYM_Arrow_Large, footprints:Snake, B.Cu at (140.1, 92.1)
- CardOutline1, CardOutline2: footprint footprints:MEC8-113-CARD-OUTLINE -> footprints:MEC8-113-CARD_2outline

Commit message: Updates
Parts:
- added R30: 1K, footprints:R_0603, F.Cu at (161.0, 97.0)
- added U3: 24LC32, footprints:DFN-8-1EP_3x2mm, F.Cu at (158.0, 97.0)
Routing:
- net /SCK: track 61.3 -> 48.0 mm
- net /~RESET: track 107.6 -> 108.8 mm

Commit message: Updates
Parts:
- moved R30 7.50 mm to (161.0, 89.5)
- moved U3 7.50 mm to (158.0, 89.5)
Routing:
- net /SCK: track 48.0 -> 61.5 mm
- net /~RESET: track 108.8 -> 121.1 mm
